File: CAD/Gold SAOs/Arista-TGS/Arista-TGS.kicad_pcb (KiCad board)
At the start: 2 copper layers, 51.9 x 34.2 mm, 7 parts

Commit message: Sao Creations
Parts:
- removed the G*** at (0.00, 0.00) (x7)
- added G*** (x7): LOGO, LOGO, F.Cu at (134.4, 73.5)
- added G***: BP LOGO, BadgePiratesLogos:BPSkull_Distressed_F.CU, B.Cu at (170.2, 93.5)
- added X1: sao_v169bis, BadgePirates:Badgelife-SAOv169-SAO_Side_B.SLK, F.Cu at (153.2, 112.0)
Routing:
- added copper zone on B.Cu, net (none)
- added copper zone on F.Cu, net (none)
Other:
- net class Default removed
- board text added: "BSides KC 2022"
