File: CAD/Gold SAOs/Corelight/Corelight SAO.kicad_pcb (KiCad board)
At the start: 2 copper layers, 60 x 60 mm, 7 parts

Commit message: Sao Creations
Parts:
- removed the G*** at (0.00, 0.00) (x7)
- added G*** (x7): LOGO, LOGO, F.Cu at (137.5, 86.2)
- added G***: BP LOGO, BadgePiratesLogos:BPSkull_Distressed_F.CU, B.Cu at (167.9, 86.7)
- added X1: sao_v169bis, BadgePirates:Badgelife-SAOv169-SAO_Side_B.SLK, F.Cu at (152.1, 115.8)
- added kibuzzard-63168605: G***, kibuzzard-63168605, B.Cu at (127.7, 102.6)
Routing:
- added copper zone on B.Cu, net (none)
- added copper zone on F.Cu, net (none)
Other:
- net class Default removed
