File: CAD/Gold SAOs/Red Canary/Red Canary.kicad_pcb (KiCad board)
At the start: 2 copper layers, 53.6 x 21.1 mm, 7 parts

Commit message: Sao Creations
Parts:
- removed the G*** at (0.00, 0.00) (x7)
- added G*** (x7): LOGO, LOGO, F.Cu at (134.9, 88.1)
- added G***: BP LOGO, BadgePiratesLogos:BPSkull_Distressed_F.CU, B.Cu at (173.1, 108.3)
- added X1: sao_v169bis, BadgePirates:Badgelife-SAOv169-SAO_Side_B.SLK, F.Cu at (132.6, 110.2)
- added kibuzzard-631686B7: G***, kibuzzard-631686B7, B.Cu at (166.1, 95.8)
Routing:
- added copper zone on B.Cu, net (none)
- added copper zone on F.Cu, net (none)
Other:
- net class Default removed
