File: CAD/Gold SAOs/Tines/Tines SAO.kicad_pcb (KiCad board)
At the start: 2 copper layers, 54.6 x 19.3 mm, 7 parts

Commit message: Sao Creations
Parts:
- removed the G*** at (0.00, 0.00) (x7)
- added G*** (x7): LOGO, LOGO, F.Cu at (134.0, 71.0)
- added G***: BP LOGO, BadgePiratesLogos:BPSkull_Distressed_F.CU, B.Cu at (131.1, 109.3)
- added X1: sao_v169bis, BadgePirates:Badgelife-SAOv169-SAO_Side_B.SLK, F.Cu at (144.3, 111.6)
- added kibuzzard-63168805: G***, kibuzzard-63168805, B.Cu at (167.2, 98.3)
Routing:
- added copper zone on B.Cu, net (none)
- added copper zone on F.Cu, net (none)
Other:
- net class Default removed
