File: CAD/BsidesKC SAO/BsidesKC 2022 Poster - Simple.kicad_pcb (KiCad board)
At the start: 2 copper layers, 39.9 x 61.6 mm, 7 parts

Commit message: soa and doc updates
Parts:
- removed the G*** at (0.00, 0.00) (x7)
- added G*** (x7): LOGO, LOGO, F.Cu at (73.8, 37.6)
- added G***: BP LOGO, BadgePiratesLogos:BPSkull_Distressed_F.CU, B.Cu at (136.4, 83.2)
- added X1: sao_v169bis, BadgePirates:Badgelife-SAOv169-SAO_Side_B.SLK, F.Cu at (151.3, 130.6)
Routing:
- added copper zone on B.Cu, net (none)
- added copper zone on F.Cu, net (none)
Other:
- net class Default removed
