File: CAD/Soldering Crew Badge/Soldering Crew Badge.kicad_pcb (KiCad board)
At the start: 2 copper layers, 75.2 x 75.2 mm, 7 parts

Commit message: Resized/Updated Soldering Village SAO
Parts:
- removed the G*** at (0.00, 0.00) (x7)
- added G*** (x7): LOGO, LOGO, F.Cu at (0.00, 0.00)
Other:
- board size 75.2 x 75.2 mm -> 50.5 x 50.6 mm

Commit message: soa and doc updates
Parts:
- removed the G*** at (0.00, 0.00) (x7)
- added D1: LED, BadgePirates:LED_Osram_Lx_P47F_D2mm_ReverseMount_Proper_Mask Only, F.Cu at (151.6, 98.7)
- added G*** (x7): LOGO, LOGO, F.Cu at (131.2, 79.4)
- added G***: BP LOGO, BadgePiratesLogos:BPSkull_Distressed_F.CU, B.Cu at (172.6, 98.2)
- added R1: 1k, BadgePirates:R_1206_3216Metric, B.Cu at (143.8, 99.3)
- added X1: sao_v169bis, BadgePirates:Badgelife-SAOv169-SAO_Side_B.SLK, F.Cu at (154.9, 124.1)
Routing:
- net GND: track 0.00 -> 27.1 mm
- net VCC: track 0.00 -> 25.7 mm
- net Net-(D1-Pad2): track 0.00 -> 5.76 mm
Other:
- outline, holes or cut-outs redrawn
- net class Default removed
